Commit message: changed pen offset

File: robots/lwr_pen.urdf (robot description, URDF)
Before this commit: robot lwr, 12 links, 11 joints
Links:
- link pen_base_link: geometry collision cylinder length=0.16 radius=0.005; visual cylinder length=0.16 radius=0.005
- link pen_ori_link: geometry visual cylinder length=0.08 radius=0.005
Joints:
- joint pen_base_joint: origin xyz=0 0 0.1 rpy=0 0 0 -> xyz=0 0 0.08 rpy=0 0 0
- joint pen_ori_joint: origin xyz=0 0 0.11 rpy=0 0 0 -> xyz=0 0 0.08 rpy=0 0 0
- joint pen_tip_joint: origin xyz=0 0 0.1 rpy=0 0 0 -> xyz=0 0 0.08 rpy=0 0 0

Commit message: added cartesian force message

File: robots/lwr_pen.urdf (robot description, URDF)
Before this commit: robot lwr, 12 links, 11 joints
Links:
- link pen_base_link: geometry collision cylinder length=0.15 radius=0.005; visual cylinder length=0.15 radius=0.005
- link pen_ori_link: geometry visual cylinder length=0.075 radius=0.005
Joints:
- joint pen_base_joint: origin xyz=0 0 0.08 rpy=0 0 0 -> xyz=0 0 0.075 rpy=0 0 0
- joint pen_ori_joint: origin xyz=0 0 0.08 rpy=0 0 0 -> xyz=0 0 0.075 rpy=0 0 0
- joint pen_tip_joint: origin xyz=0 0 0.08 rpy=0 0 0 -> xyz=0 0 0.075 rpy=0 0 0
