Commit message: fixed urdf: table size, hand orientation

File: robots/lwr_hand.urdf (robot description, URDF)
Before this commit: robot lwr, 21 links, 20 joints
Links:
- link base: geometry collision box size=.8 .85 0.04; visual box size=.7 .75 0.04
Joints:
- joint sdh_palm_joint: origin (none) -> xyz=0 0 0 rpy=0.0 0.0 -1.57079

Commit message: Updated hand urdf

File: robots/lwr_hand.urdf (robot description, URDF)
Before this commit: robot lwr, 21 links, 20 joints
Links:
- added link world_frame
Joints:
- added joint world_base_joint: type fixed, parent world_frame, child base, origin xyz=0 0 0 rpy=0 0 0
- joint base_joint: origin xyz=0 0 0.02 rpy=0 0 3.14159265359 -> xyz=0 0 0 rpy=0 0 3.14159265359
