Commit message: Updated robot frames to match KRL output

File: robots/lwr.urdf (robot description, URDF)
Before this commit: robot lwr, 9 links, 8 joints
Joints:
- joint lwr_arm_0_joint: origin xyz=0 0 0.11 rpy=0 0 0 -> xyz=0 0 0.11 rpy=0 0 3.14159265359
- joint lwr_arm_6_joint: origin xyz=0 0 0.078 rpy=0 0 0 -> xyz=0 0 0.078 rpy=0 0 3.14159265359

Commit message: Generated new URDFs

File: robots/lwr.urdf (robot description, URDF)
Before this commit: robot lwr, 9 links, 8 joints
Links:
- removed link calib_lwr_arm_base_link
- removed link world_link
- added link base, mass 2.0; collision mesh filename=package://lwr_defs/meshes/lwr/convex/arm_base_convex.stl; visual mesh filename=package://lwr_defs/meshes/lwr/base.stl
- added link world_frame; collision box size=0.7 0.75 0.04; visual box size=0.7 0.75 0.04
- link lwr_arm_1_link: geometry collision mesh filename=package://lwr_defs/meshes/lwr/convex/arm_segment_a_convex.s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; visual mesh filename=package://lwr_defs/meshes/lwr/link_1.stl
- link lwr_arm_2_link: geometry collision mesh filename=package://lwr_defs/meshes/lwr/convex/arm_segment_b_convex.s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; visual mesh filename=package://lwr_defs/meshes/lwr/link_2.stl
- link lwr_arm_3_link: geometry collision mesh filename=package://lwr_defs/meshes/lwr/convex/arm_segment_a_convex.s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; visual mesh filename=package://lwr_defs/meshes/lwr/link_3.stl
- link lwr_arm_4_link: geometry collision mesh filename=package://lwr_defs/meshes/lwr/convex/arm_segment_b_convex.s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; visual mesh filename=package://lwr_defs/meshes/lwr/link_4.stl
- link lwr_arm_5_link: geometry collision mesh filename=package://lwr_defs/meshes/lwr/convex/arm_segment_last_conve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; visual mesh filename=package://lwr_defs/meshes/lwr/link_5.stl
- link lwr_arm_6_link: geometry collision mesh filename=package://lwr_defs/meshes/lwr/convex/arm_wrist_convex.stl; visual mesh filename=package://lwr_defs/meshes/lwr/link_6.stl
- link lwr_arm_7_link: geometry collision cylinder length=0.05 radius=0.04; visual mesh filename=package://lwr_defs/meshes/lwr/link_7.stl
Joints:
- removed joint world_link_lwr_arm_base_joint
- added joint world_frame_lwr_arm_base_joint: type fixed, parent world_frame, child base, origin xyz=0 0 0 rpy=0 0 0
- joint lwr_arm_0_joint: parent calib_lwr_arm_base_link -> base
- joint lwr_arm_1_joint: origin xyz=0 0 0.2005 rpy=0 0 0 -> xyz=0 0 0.2 rpy=0 0 0

File: robots/lwr_ft_simple.urdf (robot description, URDF)
Before this commit: robot lwr, 11 links, 10 joints
Links:
- link base: geometry collision box size=0.08 0.12 0.06; collision cylinder length=0.1 radius=0.06
- link lwr_arm_1_link: geometry collision cylinder length=0.1 radius=0.06; collision sphere radius=0.06
- link lwr_arm_2_link: geometry collision cylinder length=0.1 radius=0.06; collision sphere radius=0.06
- link lwr_arm_3_link: geometry collision cylinder length=0.1 radius=0.06; collision sphere radius=0.06
- link lwr_arm_4_link: geometry collision cylinder length=0.1 radius=0.06; collision sphere radius=0.06
- link lwr_arm_5_link: geometry collision cylinder length=0.1 radius=0.06; collision sphere radius=0.06
- link lwr_arm_6_link: geometry collision sphere radius=0.07; collision sphere radius=0.07
- link lwr_arm_7_link: geometry collision cylinder length=0.05 radius=0.04; visual cylinder length=0.05 radius=0.04

File: robots/lwr_pen.urdf (robot description, URDF)
Before this commit: robot lwr, 12 links, 11 joints
Links:
- removed link lwr_arm_0_link
- added link world_frame; collision box size=0.7 0.75 0.04; visual box size=0.7 0.75 0.04
- link base: mass 50.0 -> 2.0; geometry collision mesh filename=package://lwr_defs/meshes/lwr/convex/arm_base_convex.stl; visual mesh filename=package://lwr_defs/meshes/lwr/base.stl
- link lwr_arm_1_link: geometry collision mesh filename=package://lwr_defs/meshes/lwr/convex/arm_segment_a_convex.s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; visual mesh filename=package://lwr_defs/meshes/lwr/link_1.stl
- link lwr_arm_2_link: geometry collision mesh filename=package://lwr_defs/meshes/lwr/convex/arm_segment_b_convex.s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; visual mesh filename=package://lwr_defs/meshes/lwr/link_2.stl
- link lwr_arm_3_link: geometry collision mesh filename=package://lwr_defs/meshes/lwr/convex/arm_segment_a_convex.s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; visual mesh filename=package://lwr_defs/meshes/lwr/link_3.stl
- link lwr_arm_4_link: geometry collision mesh filename=package://lwr_defs/meshes/lwr/convex/arm_segment_b_convex.s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; visual mesh filename=package://lwr_defs/meshes/lwr/link_4.stl
- link lwr_arm_5_link: geometry collision mesh filename=package://lwr_defs/meshes/lwr/convex/arm_segment_last_conve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; visual mesh filename=package://lwr_defs/meshes/lwr/link_5.stl
- link lwr_arm_6_link: geometry collision mesh filename=package://lwr_defs/meshes/lwr/convex/arm_wrist_convex.stl; visual mesh filename=package://lwr_defs/meshes/lwr/link_6.stl
- link lwr_arm_7_link: geometry collision cylinder length=0.05 radius=0.04; visual mesh filename=package://lwr_defs/meshes/lwr/link_7.stl
Joints:
- removed joint base_joint
- added joint world_frame_lwr_arm_base_joint: type fixed, parent world_frame, child base, origin xyz=0 0 0 rpy=0 0 0
- joint lwr_arm_0_joint: origin xyz=0 0 0.11 rpy=0 0 0 -> xyz=0 0 0.11 rpy=0 0 3.14159265359; parent lwr_arm_0_link -> base
- joint lwr_arm_1_joint: origin xyz=0 0 0.2005 rpy=0 0 0 -> xyz=0 0 0.2 rpy=0 0 0
- joint lwr_arm_6_joint: origin xyz=0 0 0.078 rpy=0 0 0 -> xyz=0 0 0.078 rpy=0 0 3.14159265359

File: robots/lwr_pen_simple.urdf (robot description, URDF)
Before this commit: robot lwr, 11 links, 10 joints
Links:
- removed link contact_point
- removed link force_torque_sensor
- added link pen_base_link, mass 1; collision cylinder length=0.15 radius=0.005; visual cylinder length=0.15 radius=0.005
- added link pen_ori_link, mass 1; visual cylinder length=0.075 radius=0.005
- added link pen_tip_link, mass 1; visual sphere radius=0.008
- link base: geometry collision box size=0.08 0.12 0.06; collision cylinder length=0.1 radius=0.06
- link lwr_arm_1_link: geometry collision cylinder length=0.1 radius=0.06; collision sphere radius=0.06
- link lwr_arm_2_link: geometry collision cylinder length=0.1 radius=0.06; collision sphere radius=0.06
- link lwr_arm_3_link: geometry collision cylinder length=0.1 radius=0.06; collision sphere radius=0.06
- link lwr_arm_4_link: geometry collision cylinder length=0.1 radius=0.06; collision sphere radius=0.06
- link lwr_arm_5_link: geometry collision cylinder length=0.1 radius=0.06; collision sphere radius=0.06
- link lwr_arm_6_link: geometry collision sphere radius=0.07; collision sphere radius=0.07
- link lwr_arm_7_link: geometry collision cylinder length=0.05 radius=0.04; visual cylinder length=0.05 radius=0.04
Joints:
- removed joint contact_point_joint
- removed joint force_torque_sensor_mount
- added joint pen_base_joint: type fixed, parent lwr_arm_7_link, child pen_base_link, origin xyz=0 0 0.075 rpy=0 0 0
- added joint pen_ori_joint: type fixed, parent lwr_arm_7_link, child pen_ori_link, origin xyz=0 0 0.075 rpy=0 0 0
- added joint pen_tip_joint: type fixed, parent pen_base_link, child pen_tip_link, origin xyz=0 0 0.075 rpy=0 0 0

File: robots/lwr_sdh.urdf (robot description, URDF)
Before this commit: robot lwr, 11 links, 10 joints
Links:
- removed link contact_point
- removed link force_torque_sensor
- added link sdh_finger_11_link, mass 0.1; collision mesh filename=package://schunk_description/meshes/sdh/knuckle.stl; visual mesh filename=package://schunk_description/meshes/sdh/knuckle.stl
- added link sdh_finger_12_link, mass 0.1; collision mesh filename=package://schunk_description/meshes/sdh/finger.stl; visual mesh filename=package://schunk_description/meshes/sdh/finger.stl
- added link sdh_finger_13_link, mass 0.1; collision mesh filename=package://schunk_description/meshes/sdh/finger_tip.stl; visual mesh filename=package://schunk_description/meshes/sdh/finger_tip.stl
- added link sdh_finger_21_link, mass 0.1; collision mesh filename=package://schunk_description/meshes/sdh/knuckle.stl; visual mesh filename=package://schunk_description/meshes/sdh/knuckle.stl
- added link sdh_finger_22_link, mass 0.1; collision mesh filename=package://schunk_description/meshes/sdh/finger.stl; visual mesh filename=package://schunk_description/meshes/sdh/finger.stl
- added link sdh_finger_23_link, mass 0.1; collision mesh filename=package://schunk_description/meshes/sdh/finger_tip.stl; visual mesh filename=package://schunk_description/meshes/sdh/finger_tip.stl
- added link sdh_grasp_link
- added link sdh_palm_link, mass 1; collision mesh filename=package://schunk_description/meshes/sdh/palm.stl; visual mesh filename=package://schunk_description/meshes/sdh/palm.stl
- added link sdh_thumb_1_link, mass 0.1; collision mesh filename=package://schunk_description/meshes/sdh/knuckle.stl; visual mesh filename=package://schunk_description/meshes/sdh/knuckle.stl
- added link sdh_thumb_2_link, mass 0.1; collision mesh filename=package://schunk_description/meshes/sdh/finger.stl; visual mesh filename=package://schunk_description/meshes/sdh/finger.stl
- added link sdh_thumb_3_link, mass 0.1; collision mesh filename=package://schunk_description/meshes/sdh/finger_tip.stl; visual mesh filename=package://schunk_description/meshes/sdh/finger_tip.stl
- added link sdh_tip_link
Joints:
- removed joint contact_point_joint
- removed joint force_torque_sensor_mount
- added joint sdh_finger_12_joint: type revolute, parent sdh_finger_11_link, child sdh_finger_12_link, origin xyz=0 0 0.0165 rpy=0 0 0, axis 0 1 0, limit lower=-1.570796327 upper=1.570796327 effort=100 velocity=5
- added joint sdh_finger_13_joint: type revolute, parent sdh_finger_12_link, child sdh_finger_13_link, origin xyz=0 0 0.0865 rpy=0 0 0, axis 0 1 0, limit lower=-1.570796327 upper=1.570796327 effort=100 velocity=5
- added joint sdh_finger_21_joint: type revolute, parent sdh_palm_link, child sdh_finger_21_link, origin xyz=0.01905 -0.033 0.0745 rpy=0 0 3.14159265, axis 0 0 -1, limit lower=0 upper=1.570796327 effort=100 velocity=5, mimic joint=sdh_knuckle_joint multiplier=1 offset=0
- added joint sdh_finger_22_joint: type revolute, parent sdh_finger_21_link, child sdh_finger_22_link, origin xyz=0 0 0.0165 rpy=0 0 0, axis 0 1 0, limit lower=-1.570796327 upper=1.570796327 effort=100 velocity=5
- added joint sdh_finger_23_joint: type revolute, parent sdh_finger_22_link, child sdh_finger_23_link, origin xyz=0 0 0.0865 rpy=0 0 0, axis 0 1 0, limit lower=-1.570796327 upper=1.570796327 effort=100 velocity=5
- added joint sdh_grasp_joint: type fixed, parent sdh_palm_link, child sdh_grasp_link, origin xyz=0 0 0.15 rpy=0 0 0
- added joint sdh_knuckle_joint: type revolute, parent sdh_palm_link, child sdh_finger_11_link, origin xyz=0.01905 0.033 0.0745 rpy=0 0 3.14159265, axis 0 0 1, limit lower=0 upper=1.570796327 effort=100 velocity=5
- added joint sdh_palm_joint: type fixed, parent lwr_arm_7_link, child sdh_palm_link, origin xyz=0 0 0.022 rpy=0.0 0.0 1.57079
- added joint sdh_thumb_1_joint: type fixed, parent sdh_palm_link, child sdh_thumb_1_link, origin xyz=-0.03811 0 0.0745  rpy=0 0 0
- added joint sdh_thumb_2_joint: type revolute, parent sdh_thumb_1_link, child sdh_thumb_2_link, origin xyz=0 0 0.0165 rpy=0 0 0, axis 0 1 0, limit lower=-1.570796327 upper=1.570796327 effort=100 velocity=5
- added joint sdh_thumb_3_joint: type revolute, parent sdh_thumb_2_link, child sdh_thumb_3_link, origin xyz=0 0 0.0865 rpy=0 0 0, axis 0 1 0, limit lower=-1.570796327 upper=1.570796327 effort=100 velocity=5
- added joint sdh_tip_joint: type fixed, parent sdh_palm_link, child sdh_tip_link, origin xyz=0 0 0.22 rpy=0 0 0

File: robots/lwr_simple.urdf (robot description, URDF)
Before this commit: robot lwr, 11 links, 10 joints
Links:
- removed link contact_point
- removed link force_torque_sensor
- link base: geometry collision box size=0.08 0.12 0.06; collision cylinder length=0.1 radius=0.06
- link lwr_arm_1_link: geometry collision cylinder length=0.1 radius=0.06; collision sphere radius=0.06
- link lwr_arm_2_link: geometry collision cylinder length=0.1 radius=0.06; collision sphere radius=0.06
- link lwr_arm_3_link: geometry collision cylinder length=0.1 radius=0.06; collision sphere radius=0.06
- link lwr_arm_4_link: geometry collision cylinder length=0.1 radius=0.06; collision sphere radius=0.06
- link lwr_arm_5_link: geometry collision cylinder length=0.1 radius=0.06; collision sphere radius=0.06
- link lwr_arm_6_link: geometry collision sphere radius=0.07; collision sphere radius=0.07
- link lwr_arm_7_link: geometry collision cylinder length=0.05 radius=0.04; visual cylinder length=0.05 radius=0.04
Joints:
- removed joint contact_point_joint
- removed joint force_torque_sensor_mount
