Commit message: new Kuka URDF with more accurate meshes

File: robots/lwr_sdh.urdf (robot description, URDF)
Before this commit: robot lwr, 21 links, 20 joints
Links:
- link base: geometry collision mesh filename=package://lwr_defs/meshes/lwr/convex/arm_base_convex.stl; visual mesh filename=package://lwr_defs/meshes/kuka_colour/base.obj
- link lwr_arm_1_link: geometry collision mesh filename=package://lwr_defs/meshes/lwr/convex/arm_segment_a_convex.s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; visual mesh filename=package://lwr_defs/meshes/kuka/kuka_ring.obj
- link lwr_arm_2_link: geometry collision mesh filename=package://lwr_defs/meshes/lwr/convex/arm_segment_b_convex.s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; visual mesh filename=package://lwr_defs/meshes/kuka/kuka_ring.obj
- link lwr_arm_3_link: geometry collision mesh filename=package://lwr_defs/meshes/lwr/convex/arm_segment_a_convex.s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; visual mesh filename=package://lwr_defs/meshes/kuka/kuka_ring.obj
- link lwr_arm_4_link: geometry collision mesh filename=package://lwr_defs/meshes/lwr/convex/arm_segment_b_convex.s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; visual mesh filename=package://lwr_defs/meshes/kuka/kuka_ring.obj
- link lwr_arm_5_link: geometry collision mesh filename=package://lwr_defs/meshes/lwr/convex/arm_segment_last_conve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; visual mesh filename=package://lwr_defs/meshes/kuka/kuka_ring.obj
- link lwr_arm_6_link: geometry collision mesh filename=package://lwr_defs/meshes/lwr/convex/arm_wrist_convex.stl; visual mesh filename=package://lwr_defs/meshes/kuka/kuka_wrist.obj
- link lwr_arm_7_link: geometry collision cylinder length=0.05 radius=0.04; visual mesh filename=package://lwr_defs/meshes/kuka_colour/link7.obj
