Commit message: change paths

File: urdf/defs/kuka_lwr_arm_defs.urdf.xacro (robot description, xacro)
@@ -27,5 +27,5 @@
         <origin xyz="0 0 0" rpy="0 0 ${M_PI}"/>
         <geometry>
-          <mesh filename="package://kuka_lwr4_description/meshes/kuka_colour/base.obj"/>
+          <mesh filename="package://kuka_lwr4_description/meshes/kuka_colour/base.dae"/>
         </geometry>
         <material name="Blue"/>
@@ -100,5 +100,5 @@
         <origin rpy="0 0 ${1.5*M_PI}" xyz="0 0 0.2"/>
         <geometry>
-          <mesh filename="package://kuka_lwr4_description/meshes/kuka_colour/link1.obj"/>
+          <mesh filename="package://kuka_lwr4_description/meshes/kuka_colour/link1.dae"/>
         </geometry>
         <material name="Blue"/>
@@ -107,5 +107,5 @@
         <origin rpy="0 0 ${1.5*M_PI}" xyz="0 0 0.2"/>
         <geometry>
-          <mesh filename="package://kuka_lwr4_description/meshes/kuka/link1_m.obj"/>
+          <mesh filename="package://kuka_lwr4_description/meshes/kuka_colour/link1_m.dae"/>
         </geometry>
         <material name="Grey"/>
@@ -114,5 +114,5 @@
         <origin rpy="0 0 0" xyz="0 0 0"/>
         <geometry>
-          <mesh filename="package://kuka_lwr4_description/meshes/kuka/kuka_ring.obj"/>
+          <mesh filename="package://kuka_lwr4_description/meshes/kuka_colour/kuka_ring.dae"/>
         </geometry>
         <material name="Grey"/>
@@ -202,5 +202,5 @@
         <origin rpy="0 0 ${1.5*M_PI}" xyz="0 0 0"/>
         <geometry>
-          <mesh filename="package://kuka_lwr4_description/meshes/kuka_colour/link2.obj"/>
+          <mesh filename="package://kuka_lwr4_description/meshes/kuka_colour/link2.dae"/>
         </geometry>
         <material name="Blue"/>
@@ -209,5 +209,5 @@
         <origin rpy="0 0 ${1.5*M_PI}" xyz="0 0 0"/>
         <geometry>
-          <mesh filename="package://kuka_lwr4_description/meshes/kuka/link2_m.obj"/>
+          <mesh filename="package://kuka_lwr4_description/meshes/kuka_colour/link2_m.dae"/>
         </geometry>
         <material name="Grey"/>
@@ -216,5 +216,5 @@
         <origin rpy="${0.5*M_PI} 0 0" xyz="0 0 0"/>
         <geometry>
-          <mesh filename="package://kuka_lwr4_description/meshes/kuka/kuka_ring.obj"/>
+          <mesh filename="package://kuka_lwr4_description/meshes/kuka_colour/kuka_ring.dae"/>
         </geometry>
         <material name="Grey"/>
@@ -303,5 +303,5 @@
         <origin rpy="0 0 ${1.5*M_PI}" xyz="0 0 0.2"/>
         <geometry>
-          <mesh filename="package://kuka_lwr4_description/meshes/kuka_colour/link3.obj"/>
+          <mesh filename="package://kuka_lwr4_description/meshes/kuka_colour/link3.dae"/>
         </geometry>
         <material name="Blue"/>
@@ -310,5 +310,5 @@
         <origin rpy="0 0 ${1.5*M_PI}" xyz="0 0 0.2"/>
         <geometry>
-          <mesh filename="package://kuka_lwr4_description/meshes/kuka/link3_m.obj"/>
+          <mesh filename="package://kuka_lwr4_description/meshes/kuka_colour/link3_m.dae"/>
         </geometry>
         <material name="Grey"/>
@@ -317,5 +317,5 @@
         <origin rpy="0 0 0" xyz="0 0 0"/>
         <geometry>
-          <mesh filename="package://kuka_lwr4_description/meshes/kuka/kuka_ring.obj"/>
+          <mesh filename="package://kuka_lwr4_description/meshes/kuka_colour/kuka_ring.dae"/>
         </geometry>
         <material name="Grey"/>
@@ -405,5 +405,5 @@
         <origin rpy="0 0 ${1.5*M_PI}" xyz="0 0 0"/>
         <geometry>
-          <mesh filename="package://kuka_lwr4_description/meshes/kuka_colour/link4.obj"/>
+          <mesh filename="package://kuka_lwr4_description/meshes/kuka_colour/link4.dae"/>
         </geometry>
         <material name="Blue"/>
@@ -412,5 +412,5 @@
         <origin rpy="0 0 ${1.5*M_PI}" xyz="0 0 0"/>
         <geometry>
-          <mesh filename="package://kuka_lwr4_description/meshes/kuka/link4_m.obj"/>
+          <mesh filename="package://kuka_lwr4_description/meshes/kuka_colour/link4_m.dae"/>
         </geometry>
         <material name="Grey"/>
@@ -419,5 +419,5 @@
         <origin rpy="${0.5*M_PI} 0 0" xyz="0 0 0"/>
         <geometry>
-          <mesh filename="package://kuka_lwr4_description/meshes/kuka/kuka_ring.obj"/>
+          <mesh filename="package://kuka_lwr4_description/meshes/kuka_colour/kuka_ring.dae"/>
         </geometry>
         <material name="Grey"/>
@@ -506,5 +506,5 @@
         <origin rpy="0 0 ${1.5*M_PI}" xyz="0 0 0.19"/>
         <geometry name="${name}_arm_5_geom">
-          <mesh filename="package://kuka_lwr4_description/meshes/kuka_colour/link5.obj"/>
+          <mesh filename="package://kuka_lwr4_description/meshes/kuka_colour/link5.dae"/>
         </geometry>
         <material name="Blue"/>
@@ -513,5 +513,5 @@
         <origin rpy="0 0 0" xyz="0 0 0"/>
         <geometry>
-          <mesh filename="package://kuka_lwr4_description/meshes/kuka/kuka_ring.obj"/>
+          <mesh filename="package://kuka_lwr4_description/meshes/kuka_colour/kuka_ring.dae"/>
         </geometry>
         <material name="Grey"/>
@@ -600,5 +600,5 @@
         <origin rpy="0 0 ${M_PI}" xyz="0 0 0"/>
         <geometry>
-          <mesh filename="package://kuka_lwr4_description/meshes/kuka/kuka_wrist.obj"/>
+          <mesh filename="package://kuka_lwr4_description/meshes/kuka_colour/kuka_wrist.dae"/>
         </geometry>
         <material name="Grey"/>
@@ -680,5 +680,5 @@
         <origin xyz="0 0 0" rpy="0 0 0"/>
         <geometry>
-          <mesh filename="package://kuka_lwr4_description/meshes/kuka_colour/link7.obj"/>
+          <mesh filename="package://kuka_lwr4_description/meshes/kuka_colour/link7.dae"/>
         </geometry>
         <material name="Grey"/>

File: urdf/lwr_robotiq_3finger.urdf.xacro (robot description, xacro)
@@ -54,5 +54,5 @@
       <origin rpy="${0.5*M_PI} 0 0"/>
       <geometry>
-        <mesh filename="package://kuka_lwr4_description/meshes/robotiq/AGS-CPL-175_20171219.obj"/>
+        <mesh filename="package://kuka_lwr4_description/meshes/robotiq/AGS-CPL-175_20171219.dae"/>
       </geometry>
       <material name="gray">
