Commit message: Rename world_frame to table to avoid clash with EXOTica naming - Exotica uses world_frame as a virtual frame name (from SRDF) thus having it here for a table causes a conflict. Now named as what it should be - table.

File: urdf/lwr.urdf.xacro (robot description, xacro)
@@ -10,5 +10,5 @@
   </xacro:if>
   <xacro:include filename="$(find kuka_lwr4_description)/urdf/defs/materials.xml"/>
-  <link name="world_frame">
+  <link name="table">
       <visual>
         <origin xyz="0 0 -0.02" rpy="0 0 0"/>
@@ -25,5 +25,5 @@
       </collision>
   </link>
-  <kuka_lwr_arm parent="world_frame" name="lwr" right="1" gazebo="$(arg use_gazebo)" transmission="$(arg use_transmission)" collisionsimple="$(arg collision_simple)" visualsimple="$(arg visual_simple)">
+  <kuka_lwr_arm parent="table" name="lwr" right="1" gazebo="$(arg use_gazebo)" transmission="$(arg use_transmission)" collisionsimple="$(arg collision_simple)" visualsimple="$(arg visual_simple)">
     <origin xyz="0 0 0" rpy="0 0 0"/>
   </kuka_lwr_arm>

Commit message: fix tabsize

File: urdf/lwr.urdf.xacro (robot description, xacro)
@@ -11,17 +11,17 @@
   <xacro:include filename="$(find kuka_lwr4_description)/urdf/defs/materials.xml"/>
   <link name="table">
-      <visual>
-        <origin xyz="0 0 -0.02" rpy="0 0 0"/>
-        <geometry>
-          <box size="0.7 0.75 0.04"/>
-        </geometry>
-        <material name="DarkGrey"/>
-      </visual>
-      <collision>
-        <origin xyz="0 0 -0.02" rpy="0 0 0"/>
-        <geometry>
-          <box size="0.7 0.75 0.04"/>
-        </geometry>
-      </collision>
+    <visual>
+      <origin xyz="0 0 -0.02" rpy="0 0 0"/>
+      <geometry>
+        <box size="0.7 0.75 0.04"/>
+      </geometry>
+      <material name="DarkGrey"/>
+    </visual>
+    <collision>
+      <origin xyz="0 0 -0.02" rpy="0 0 0"/>
+      <geometry>
+        <box size="0.7 0.75 0.04"/>
+      </geometry>
+    </collision>
   </link>
   <kuka_lwr_arm parent="table" name="lwr" right="1" gazebo="$(arg use_gazebo)" transmission="$(arg use_transmission)" collisionsimple="$(arg collision_simple)" visualsimple="$(arg visual_simple)">

Commit message: change table colour to brown

File: urdf/lwr.urdf.xacro (robot description, xacro)
@@ -16,5 +16,8 @@
         <box size="0.7 0.75 0.04"/>
       </geometry>
-      <material name="DarkGrey"/>
+      <material name="table_brown">
+        <!-- wooden brown table -->
+        <color rgba="0.839215686 0.694117647 0.42745098 1.0"/>
+      </material>
     </visual>
     <collision>

Commit message: wood texture for Gazebo

File: urdf/lwr.urdf.xacro (robot description, xacro)
@@ -28,4 +28,10 @@
     </collision>
   </link>
+  <xacro:if value="$(arg use_gazebo)">
+  <gazebo reference="table">
+    <!-- Gazebo wood texture -->
+    <material>Gazebo/Wood</material>
+  </gazebo>
+  </xacro:if>
   <kuka_lwr_arm parent="table" name="lwr" right="1" gazebo="$(arg use_gazebo)" transmission="$(arg use_transmission)" collisionsimple="$(arg collision_simple)" visualsimple="$(arg visual_simple)">
     <origin xyz="0 0 0" rpy="0 0 0"/>
